File: hardware/hackrf-one/baseband.sch (KiCad schematic (older format))
At the start: 136 parts, among them P14 XCVR_CLKOUT, P15 INTR, P16 CLKIN, P18 OEB, P2 CLKOUT, P36 VAA, P37 SCL, P38 SDA, P39 SSP1_SCK, P40 SSP1_MOSI, P41 SSP1_MISO, P53 CS_XCVR, P54 CS_AD, P55 TXENABLE, P56 RXENABLE, P57 XTAL2, P58 GCK1, P59 GCK2, P60 SGPIO_CLK, P61 DA0, P62 DA7, P63 DD0, P64 DD9, P65 DA4, P66 DD5, P67 RSSI, P83 GND, P84 GND, P85 GND, P86 GND, P87 GND, P88 GND, P89 GND, P9 BASEBAND, P90 GND, P91 GND, P92 GND, Q3 MOSFET_P, T3 RX_BALUN, T4 TX_BALUN, U17 MAX2837, U18 MAX5864, U19 SI5351C, X1 GSG-XTAL4PIN

Commit message: HackRF One: replaced NRND GRM155R61A104KA01D 100 nF capacitors with GCM155R71C104KA55
Parts:
- C113, C119, C120, C121, C122, C123, C167, C71, C73, C75, C77, C79, C81, C83, C91: Description CAP CER 0.1UF 10V 10% X5R 0402 -> CAP CER 0.1UF 16V 10% X7R 0402; Part Number GRM155R61A104KA01D -> GCM155R71C104KA55
Changed lines of the file:
@@
 F 3 "" H 3450 1250 60  0001 C CNN
 F 4 "Murata" H 3450 1250 60  0001 C CNN "Manufacturer"
-F 5 "GRM155R61A104KA01D" H 3450 1250 60  0001 C CNN "Part Number"
-F 6 "CAP CER 0.1UF 10V 10% X5R 0402" H 3450 1250 60  0001 C CNN "Description"
+F 5 "GCM155R71C104KA55" H 3450 1250 60  0001 C CNN "Part Number"
+F 6 "CAP CER 0.1UF 16V 10% X7R 0402" H 3450 1250 60  0001 C CNN "Description"
 	1    3450 1250
 	1    0    0    -1
@@
 F 3 "" H 15550 1200 60  0001 C CNN
 F 4 "Murata" H 15550 1200 60  0001 C CNN "Manufacturer"
-F 5 "GRM155R61A104KA01D" H 15550 1200 60  0001 C CNN "Part Number"
-F 6 "CAP CER 0.1UF 10V 10% X5R 0402" H 15550 1200 60  0001 C CNN "Description"
+F 5 "GCM155R71C104KA55" H 15550 1200 60  0001 C CNN "Part Number"
+F 6 "CAP CER 0.1UF 16V 10% X7R 0402" H 15550 1200 60  0001 C CNN "Description"
 	1    15550 1200
 	1    0    0    -1
@@
 F 3 "" H 14950 1200 60  0001 C CNN
 F 4 "Murata" H 14950 1200 60  0001 C CNN "Manufacturer"
-F 5 "GRM155R61A104KA01D" H 14950 1200 60  0001 C CNN "Part Number"
-F 6 "CAP CER 0.1UF 10V 10% X5R 0402" H 14950 1200 60  0001 C CNN "Description"
+F 5 "GCM155R71C104KA55" H 14950 1200 60  0001 C CNN "Part Number"
+F 6 "CAP CER 0.1UF 16V 10% X7R 0402" H 14950 1200 60  0001 C CNN "Description"
 	1    14950 1200
 	1    0    0    -1
@@
 F 3 "" H 14350 1200 60  0001 C CNN
 F 4 "Murata" H 14350 1200 60  0001 C CNN "Manufacturer"
-F 5 "GRM155R61A104KA01D" H 14350 1200 60  0001 C CNN "Part Number"
-F 6 "CAP CER 0.1UF 10V 10% X5R 0402" H 14350 1200 60  0001 C CNN "Description"
+F 5 "GCM155R71C104KA55" H 14350 1200 60  0001 C CNN "Part Number"
+F 6 "CAP CER 0.1UF 16V 10% X7R 0402" H 14350 1200 60  0001 C CNN "Description"
 	1    14350 1200
 	1    0    0    -1
@@
 F 3 "" H 13750 1200 60  0001 C CNN
 F 4 "Murata" H 13750 1200 60  0001 C CNN "Manufacturer"
-F 5 "GRM155R61A104KA01D" H 13750 1200 60  0001 C CNN "Part Number"
-F 6 "CAP CER 0.1UF 10V 10% X5R 0402" H 13750 1200 60  0001 C CNN "Description"
+F 5 "GCM155R71C104KA55" H 13750 1200 60  0001 C CNN "Part Number"
+F 6 "CAP CER 0.1UF 16V 10% X7R 0402" H 13750 1200 60  0001 C CNN "Description"
 	1    13750 1200
 	1    0    0    -1
@@
 F 3 "" H 13150 1200 60  0001 C CNN
 F 4 "Murata" H 13150 1200 60  0001 C CNN "Manufacturer"
-F 5 "GRM155R61A104KA01D" H 13150 1200 60  0001 C CNN "Part Number"
-F 6 "CAP CER 0.1UF 10V 10% X5R 0402" H 13150 1200 60  0001 C CNN "Description"
+F 5 "GCM155R71C104KA55" H 13150 1200 60  0001 C CNN "Part Number"
+F 6 "CAP CER 0.1UF 16V 10% X7R 0402" H 13150 1200 60  0001 C CNN "Description"
 	1    13150 1200
 	1    0    0    -1
@@
 F 3 "" H 12550 1200 60  0001 C CNN
 F 4 "Murata" H 12550 1200 60  0001 C CNN "Manufacturer"
-F 5 "GRM155R61A104KA01D" H 12550 1200 60  0001 C CNN "Part Number"
-F 6 "CAP CER 0.1UF 10V 10% X5R 0402" H 12550 1200 60  0001 C CNN "Description"
+F 5 "GCM155R71C104KA55" H 12550 1200 60  0001 C CNN "Part Number"
+F 6 "CAP CER 0.1UF 16V 10% X7R 0402" H 12550 1200 60  0001 C CNN "Description"
 	1    12550 1200
 	1    0    0    -1
@@
 F 3 "" H 11950 1200 60  0001 C CNN
 F 4 "Murata" H 11950 1200 60  0001 C CNN "Manufacturer"
-F 5 "GRM155R61A104KA01D" H 11950 1200 60  0001 C CNN "Part Number"
-F 6 "CAP CER 0.1UF 10V 10% X5R 0402" H 11950 1200 60  0001 C CNN "Description"
+F 5 "GCM155R71C104KA55" H 11950 1200 60  0001 C CNN "Part Number"
+F 6 "CAP CER 0.1UF 16V 10% X7R 0402" H 11950 1200 60  0001 C CNN "Description"
 	1    11950 1200
 	1    0    0    -1
@@
 F 3 "" H 15300 7500 60  0001 C CNN
 F 4 "Murata" H 15300 7500 60  0001 C CNN "Manufacturer"
-F 5 "GRM155R61A104KA01D" H 15300 7500 60  0001 C CNN "Part Number"
-F 6 "CAP CER 0.1UF 10V 10% X5R 0402" H 15300 7500 60  0001 C CNN "Description"
+F 5 "GCM155R71C104KA55" H 15300 7500 60  0001 C CNN "Part Number"
+F 6 "CAP CER 0.1UF 16V 10% X7R 0402" H 15300 7500 60  0001 C CNN "Description"
 	1    15300 7500
 	1    0    0    -1
@@
 F 3 "" H 2300 10000 60  0001 C CNN
 F 4 "Murata" H 2300 10000 60  0001 C CNN "Manufacturer"
-F 5 "GRM155R61A104KA01D" H 2300 10000 60  0001 C CNN "Part Number"
-F 6 "CAP CER 0.1UF 10V 10% X5R 0402" H 2300 10000 60  0001 C CNN "Description"
+F 5 "GCM155R71C104KA55" H 2300 10000 60  0001 C CNN "Part Number"
+F 6 "CAP CER 0.1UF 16V 10% X7R 0402" H 2300 10000 60  0001 C CNN "Description"
 	1    2300 10000
 	1    0    0    -1
@@
 F 3 "" H 1900 10000 60  0001 C CNN
 F 4 "Murata" H 1900 10000 60  0001 C CNN "Manufacturer"
-F 5 "GRM155R61A104KA01D" H 1900 10000 60  0001 C CNN "Part Number"
-F 6 "CAP CER 0.1UF 10V 10% X5R 0402" H 1900 10000 60  0001 C CNN "Description"
+F 5 "GCM155R71C104KA55" H 1900 10000 60  0001 C CNN "Part Number"
+F 6 "CAP CER 0.1UF 16V 10% X7R 0402" H 1900 10000 60  0001 C CNN "Description"
 	1    1900 10000
 	1    0    0    -1
@@
 F 3 "" H 1500 10000 60  0001 C CNN
 F 4 "Murata" H 1500 10000 60  0001 C CNN "Manufacturer"
-F 5 "GRM155R61A104KA01D" H 1500 10000 60  0001 C CNN "Part Number"
-F 6 "CAP CER 0.1UF 10V 10% X5R 0402" H 1500 10000 60  0001 C CNN "Description"
+F 5 "GCM155R71C104KA55" H 1500 10000 60  0001 C CNN "Part Number"
+F 6 "CAP CER 0.1UF 16V 10% X7R 0402" H 1500 10000 60  0001 C CNN "Description"
 	1    1500 10000
 	1    0    0    -1
@@
 F 3 "" H 1100 10000 60  0001 C CNN
 F 4 "Murata" H 1100 10000 60  0001 C CNN "Manufacturer"
-F 5 "GRM155R61A104KA01D" H 1100 10000 60  0001 C CNN "Part Number"
-F 6 "CAP CER 0.1UF 10V 10% X5R 0402" H 1100 10000 60  0001 C CNN "Description"
+F 5 "GCM155R71C104KA55" H 1100 10000 60  0001 C CNN "Part Number"
+F 6 "CAP CER 0.1UF 16V 10% X7R 0402" H 1100 10000 60  0001 C CNN "Description"
 	1    1100 10000
 	1    0    0    -1
@@
 F 3 "" H 3800 6850 60  0001 C CNN
 F 4 "Murata" H 3800 6850 60  0001 C CNN "Manufacturer"
-F 5 "GRM155R61A104KA01D" H 3800 6850 60  0001 C CNN "Part Number"
-F 6 "CAP CER 0.1UF 10V 10% X5R 0402" H 3800 6850 60  0001 C CNN "Description"
+F 5 "GCM155R71C104KA55" H 3800 6850 60  0001 C CNN "Part Number"
+F 6 "CAP CER 0.1UF 16V 10% X7R 0402" H 3800 6850 60  0001 C CNN "Description"
 	1    3800 6850
 	1    0    0    -1
@@
 F 3 "" H 1600 2550 60  0001 C CNN
 F 4 "Murata" H 1600 2550 60  0001 C CNN "Manufacturer"
-F 5 "GRM155R61A104KA01D" H 1600 2550 60  0001 C CNN "Part Number"
-F 6 "CAP CER 0.1UF 10V 10% X5R 0402" H 1600 2550 60  0001 C CNN "Description"
+F 5 "GCM155R71C104KA55" H 1600 2550 60  0001 C CNN "Part Number"
+F 6 "CAP CER 0.1UF 16V 10% X7R 0402" H 1600 2550 60  0001 C CNN "Description"
 	1    1600 2550
 	1    0    0    -1

Commit message: HackRF One: replaced NRND GRM1555C1H330JA01D 33 pF capacitors with GCM1555C1H330JA16
Parts:
- C115: Part Number GRM1555C1H330JA01D -> GCM1555C1H330JA16
Changed lines of the file:
@@
 F 3 "" H 6700 7050 60  0001 C CNN
 F 4 "Murata" H 18050 9300 60  0001 C CNN "Manufacturer"
-F 5 "GRM1555C1H330JA01D" H 18050 9300 60  0001 C CNN "Part Number"
+F 5 "GCM1555C1H330JA16" H 18050 9300 60  0001 C CNN "Part Number"
 F 6 "CAP CER 33PF 50V 5% NP0 0402" H 18050 9300 60  0001 C CNN "Description"
 	1    6700 7050

Commit message: HackRF One: replaced EoL GRM21BR61A106KE19L 10 uF capacitors with GRM21BR61C106KE15
Parts:
- C105: Description CAP CER 10UF 10V 10% X5R 0805 -> CAP CER 10UF 16V 10% X5R 0805; Part Number GRM21BR61A106KE19L -> GRM21BR61C106KE15
Changed lines of the file:
@@
 F 3 "" H 2000 4150 60  0001 C CNN
 F 4 "Murata" H 2000 4150 60  0001 C CNN "Manufacturer"
-F 5 "GRM21BR61A106KE19L" H 2000 4150 60  0001 C CNN "Part Number"
-F 6 "CAP CER 10UF 10V 10% X5R 0805" H 2000 4150 60  0001 C CNN "Description"
+F 5 "GRM21BR61C106KE15" H 2000 4150 60  0001 C CNN "Part Number"
+F 6 "CAP CER 10UF 16V 10% X5R 0805" H 2000 4150 60  0001 C CNN "Description"
 	1    2000 4150
 	1    0    0    -1

Commit message: HackRF One: replaced obsolete LXES15AAA1-100 TVS diode with LXES15AAA1-153
Parts:
- D3, D9: Part Number LXES15AAA1-100 -> LXES15AAA1-153
Changed lines of the file:
@@
 F 3 "" H 5700 9950 60  0001 C CNN
 F 4 "Murata" H 5700 9950 60  0001 C CNN "Manufacturer"
-F 5 "LXES15AAA1-100" H 5700 9950 60  0001 C CNN "Part Number"
+F 5 "LXES15AAA1-153" H 5700 9950 60  0001 C CNN "Part Number"
 F 6 "TVS DIODE ESD .05PF 15KV 0402" H 5700 9950 60  0001 C CNN "Description"
 	1    5700 9950
@@
 F 3 "" H 3400 9200 60  0001 C CNN
 F 4 "Murata" H 3400 9200 60  0001 C CNN "Manufacturer"
-F 5 "LXES15AAA1-100" H 3400 9200 60  0001 C CNN "Part Number"
+F 5 "LXES15AAA1-153" H 3400 9200 60  0001 C CNN "Part Number"
 F 6 "TVS DIODE ESD .05PF 15KV 0402" H 3400 9200 60  0001 C CNN "Description"
 	1    3400 9200

Commit message: HackRF One: prefer Murata balun for T3 and T4
Parts:
- T3: Manufacturer Johanson Technology -> Murata; Note: Alternative part: Murata LDB182G4510G-120 -> Alternative part: Johanson Technology 2500BL14M100T; Part Number 2500BL14M100T -> LDB182G4510G-120
- T4: Manufacturer Johanson Technology -> Murata; Note Alternative part: Murata LDB182G4510G-120 -> Alternative part: Johanson Technology 2500BL14M100T; Part Number 2500BL14M100T -> LDB182G4510G-120
Changed lines of the file:
@@
 F 2 "hackrf:GSG-2500BL14M100" H 4750 5600 60  0001 C CNN
 F 3 "" H 4750 5600 60  0001 C CNN
-F 4 "Johanson Technology" H 4750 5600 60  0001 C CNN "Manufacturer"
-F 5 "2500BL14M100T" H 4750 5600 60  0001 C CNN "Part Number"
+F 4 "Murata" H 4750 5600 60  0001 C CNN "Manufacturer"
+F 5 "LDB182G4510G-120" H 4750 5600 60  0001 C CNN "Part Number"
 F 6 "BALUN CERAMIC CHIP WIMAX 2.5GHZ" H 4750 5600 60  0001 C CNN "Description"
-F 7 "Alternative part: Murata LDB182G4510G-120" H 4750 5600 60  0001 C CNN "Note"
+F 7 "Alternative part: Johanson Technology 2500BL14M100T" H 4750 5600 60  0001 C CNN "Note"
 	1    4750 5600
 	-1   0    0    1
@@
 F 2 "hackrf:GSG-2500BL14M100" H 4750 4500 60  0001 C CNN
 F 3 "" H 4750 4500 60  0001 C CNN
-F 4 "Johanson Technology" H 4750 4500 60  0001 C CNN "Manufacturer"
-F 5 "2500BL14M100T" H 4750 4500 60  0001 C CNN "Part Number"
+F 4 "Murata" H 4750 4500 60  0001 C CNN "Manufacturer"
+F 5 "LDB182G4510G-120" H 4750 4500 60  0001 C CNN "Part Number"
 F 6 "BALUN CERAMIC CHIP WIMAX 2.5GHZ" H 4750 4500 60  0001 C CNN "Description"
-F 7 "Alternative part: Murata LDB182G4510G-120" H 4750 4500 60  0001 C CNN "Note:"
+F 7 "Alternative part: Johanson Technology 2500BL14M100T" H 4750 4500 60  0001 C CNN "Note:"
 	1    4750 4500
 	-1   0    0    1
