File: hardware/hackrf-one/baseband.sch (KiCad schematic (older format))
At the start: 136 parts, among them P14 XCVR_CLKOUT, P15 INTR, P16 CLKIN, P18 OEB, P2 CLKOUT, P36 VAA, P37 SCL, P38 SDA, P39 SSP1_SCK, P40 SSP1_MOSI, P41 SSP1_MISO, P53 CS_XCVR, P54 CS_AD, P55 TXENABLE, P56 RXENABLE, P57 XTAL2, P58 GCK1, P59 GCK2, P60 SGPIO_CLK, P61 DA0, P62 DA7, P63 DD0, P64 DD9, P65 DA4, P66 DD5, P67 RSSI, P83 GND, P84 GND, P85 GND, P86 GND, P87 GND, P88 GND, P89 GND, P9 BASEBAND, P90 GND, P91 GND, P92 GND, Q3 MOSFET_P, T3 RX_BALUN, T4 TX_BALUN, U17 MAX2837, U18 MAX5864, U19 SI5351C, X1 GSG-XTAL4PIN

Commit message: HackRF One: replaced various capacitors that are NRND
Parts:
- C100, C97, C98: Manufacturer Murata -> Samsung; Part Number GRM155R61A334KE15D -> CL05A334KP5NNN
- C101, C102, C103, C107, C108, C109, C110, C84, C85, C86, C94, C95, C96, C99: Manufacturer Murata -> Samsung; Part Number GRM1555C1H220JA01D -> CL05C220JB5NNN
- C104, C111: Manufacturer Murata -> Samsung; Part Number GRM1555C1H3R0CA01D -> CL05C030CB5NNN
- C112: Manufacturer Murata -> Samsung; Part Number GRM1555C1H181JA01D -> CL05C181JB5NNN
- C114: Manufacturer Murata -> Samsung; Part Number GRM155R71H332KA01D -> CL05B332KB5NNN
- C116: Part Number GRM1555C1H470JA01D -> GCM1555C1H470JA16
- C159, C165, C168, C68, C69, C90: Part Number GRM1555C1H101JA01D -> GCM1555C1H101JA16
- C169, C170: Part Number GRM1555C1E1R8BA01D -> GJM1555C1H1R8CB01
- C87, C88, C89, C92, C93: Description CAP CER 10000PF 16V 10% X7R 0402 -> CAP CER 10000PF 50V 10% X7R 0402; Part Number GRM155R71C103KA01D -> GCM155R71H103KA55
