File: hardware/hackrf-one/baseband.sch (KiCad schematic (older format))
At the start: 136 parts, among them P14 XCVR_CLKOUT, P15 INTR, P16 CLKIN, P18 OEB, P2 CLKOUT, P37 SCL, P38 SDA, P39 SSP1_SCK, P40 SSP1_COPI, P41 SSP1_CIPO, P53 CS_XCVR, P54 CS_AD, P55 TXENABLE, P56 RXENABLE, P57 XTAL2, P58 GCK1, P59 GCK2, P60 SGPIO_CLK, P61 DA0, P62 DA7, P63 DD0, P64 DD9, P65 DA4, P66 DD5, P67 RSSI, P83 GND, P84 GND, P85 GND, P86 GND, P87 GND, P88 GND, P89 GND, P9 BASEBAND, P90 GND, P91 GND, P92 GND, Q3 MOSFET_P, T3 RX_BALUN, T4 TX_BALUN, U17 MAX2837, U18 MAX5864, U19 SI5351C, X1 GSG-XTAL4PIN

Commit message: HackRF One: add ADC pin straps for hardware version detection
update power supply schematic symbols
Other:
- moved on the sheet: R105
