File: hardware/hackrf-one/frontend.sch (KiCad schematic (older format))
At the start: 144 parts, among them J10 GND_CLIP, J2 RF-SHIELD-FRAME, J3 RF-SHIELD-COVER, J4 MOUNTING_HOLE, J5 MOUNTING_HOLE, J6 MOUNTING_HOLE, J7 MOUNTING_HOLE, J8 MOUNTING_HOLE, J9 MOUNTING_HOLE, P13 GPO1, P17 GPO6, P19 GPO3, P21 REF_IN, P27 MIXER_SDATA, P31 MIXER_SCLK, P32 MIXER_ENX, P33 MIXER_RESETX, P34 MIX_BYPASS, P35 !MIX_BYPASS, P4 ANTENNA, P43 RX, P44 HP, P45 LP, P46 TX_MIX_BP, P47 RX_MIX_BP, P48 TX_AMP, P49 RX_AMP, P50 AMP_BYPASS, P51 !TX_AMP_PWR, P52 !RX_AMP_PWR, P6 GPO4, P7 GPO2, T1 MIX_IN_BALUN, T2 MIX_OUT_BALUN, U1 SKY13453, U10 SKY13453, U11 SKY13453, U12 SKY13317, U13 TRF37D73, U14 SKY13317, U16 AP2553W6-7, U2 SKY13453, U25 TRF37A73, U3 RX_LOWPASS_FILTER, U4 RFFC5072, U5 SKY13453, U6 SKY13453, U7 SKY13453, U8 RX_HIGHPASS_FILTER, U9 SKY13317

Commit message: HackRF One: updated layout to match recent changes to schematic
Parts:
- U13, U25: footprint (none) -> gsg-modules:WSON8
- U16: footprint (none) -> gsg-modules:SOT457
Changed lines of the file:
@@
 F 0 "U25" H 13000 5850 60  0000 C CNN
 F 1 "TRF37A73" H 13000 6150 60  0000 C CNN
-F 2 "" H 13000 6000 60  0001 C CNN
+F 2 "gsg-modules:WSON8" H 13000 6000 60  0001 C CNN
 F 3 "" H 13000 6000 60  0001 C CNN
 F 4 "Texas Instruments" H 13000 5900 60  0001 C CNN "Manufacturer"
@@
 F 0 "U13" H 9400 9200 60  0000 C CNN
 F 1 "TRF37D73" H 9400 9500 60  0000 C CNN
-F 2 "" H 9400 9350 60  0001 C CNN
+F 2 "gsg-modules:WSON8" H 9400 9350 60  0001 C CNN
 F 3 "" H 9400 9350 60  0001 C CNN
 F 4 "Texas Instruments" H 9400 9250 60  0001 C CNN "Manufacturer"
@@
 F 0 "U16" H 15450 7400 60  0000 C CNN
 F 1 "AP2553W6-7" H 15450 6900 60  0000 C CNN
-F 2 "" H 15450 7150 60  0000 C CNN
+F 2 "gsg-modules:SOT457" H 15450 7150 60  0001 C CNN
 F 3 "" H 15450 7150 60  0000 C CNN
 F 4 "Diodes Inc." H 15450 7150 60  0001 C CNN "Manufacturer"

Commit message: HackRF One: replaced various capacitors that are NRND
Parts:
- C10, C16, C162, C163, C19, C2, C22, C30, C4, C54, C56, C6: Description CAP CER 10000PF 16V 10% X7R 0402 -> CAP CER 10000PF 50V 10% X7R 0402; Part Number GRM155R71C103KA01D -> GCM155R71H103KA55
- C12, C13: Manufacturer Murata -> Samsung; Part Number GRM155R71H331KA01D -> CL05B331KB5NNN
- C15: Manufacturer Murata -> Samsung; Part Number GRM1555C1H181JA01D -> CL05C181JB5NNN
- C160, C41, C42, C52, C70: Part Number GRM1555C1H101JA01D -> GCM1555C1H101JA16
- C21, C32, C43, C48, C51, C8: Manufacturer Murata -> Samsung; Part Number GRM1555C1H220JA01D -> CL05C220JB5NNN
- C26, C27: Part Number GRM1555C1H470JA01D -> GCM1555C1H470JA16
