File: hardware/hackrf-one/frontend.sch (KiCad schematic (older format))
At the start: 144 parts, among them J10 GND_CLIP, J2 RF-SHIELD-FRAME, J3 RF-SHIELD-COVER, J4 MOUNTING_HOLE, J5 MOUNTING_HOLE, J6 MOUNTING_HOLE, J7 MOUNTING_HOLE, J8 MOUNTING_HOLE, J9 MOUNTING_HOLE, P13 GPO1, P17 GPO6, P19 GPO3, P21 REF_IN, P27 MIXER_SDATA, P31 MIXER_SCLK, P32 MIXER_ENX, P33 MIXER_RESETX, P34 MIX_BYPASS, P35 !MIX_BYPASS, P4 ANTENNA, P42 TX, P43 RX, P44 HP, P45 LP, P46 TX_MIX_BP, P47 RX_MIX_BP, P48 TX_AMP, P49 RX_AMP, P50 AMP_BYPASS, P51 !TX_AMP_PWR, P52 !RX_AMP_PWR, P6 GPO4, P7 GPO2, Q1 MOSFET_P, Q2 MOSFET_P, Q4 MOSFET_P, T1 MIX_IN_BALUN, T2 MIX_OUT_BALUN, U1 SKY13350, U10 SKY13350, U11 SKY13350, U12 SKY13317, U13 MGA-81563, U14 SKY13317, U2 SKY13350, U25 MGA-81563, U3 RX_LOWPASS_FILTER, U4 RFFC5072, U5 SKY13350, U6 SKY13350, U7 SKY13350, U8 RX_HIGHPASS_FILTER, U9 SKY13317

Commit message: HackRF One: add ADC pin straps for hardware version detection
update power supply schematic symbols
Changed lines of the file:
@@
 $EndComp
 $Comp
-L power:VAA #PWR04
-U 1 1 50457D5F
-P 12300 6100
-F 0 "#PWR04" H 12300 6160 30  0001 C CNN
-F 1 "VAA" H 12300 6210 30  0000 C CNN
-F 2 "" H 12300 6100 60  0001 C CNN
-F 3 "" H 12300 6100 60  0001 C CNN
-	1    12300 6100
-	1    0    0    -1
-$EndComp
-$Comp
 L power:GND #PWR05
 U 1 1 50457CD5
@@
 MIX_CLK
 $Comp
-L power:VAA #PWR013
-U 1 1 5043D020
-P 10500 7900
-F 0 "#PWR013" H 10500 7960 30  0001 C CNN
-F 1 "VAA" H 10500 8010 30  0000 C CNN
-F 2 "" H 10500 7900 60  0001 C CNN
-F 3 "" H 10500 7900 60  0001 C CNN
-	1    10500 7900
-	1    0    0    -1
-$EndComp
-$Comp
-L power:VAA #PWR014
-U 1 1 5043CFFC
-P 5650 7950
-F 0 "#PWR014" H 5650 8010 30  0001 C CNN
-F 1 "VAA" H 5650 8060 30  0000 C CNN
-F 2 "" H 5650 7950 60  0001 C CNN
-F 3 "" H 5650 7950 60  0001 C CNN
-	1    5650 7950
-	1    0    0    -1
-$EndComp
-$Comp
 L power:GND #PWR015
 U 1 1 5043CFF1
@@
 $EndComp
 $Comp
-L power:VAA #PWR016
-U 1 1 5043CF9A
-P 6600 3050
-F 0 "#PWR016" H 6600 3110 30  0001 C CNN
-F 1 "VAA" H 6600 3160 30  0000 C CNN
-F 2 "" H 6600 3050 60  0001 C CNN
-F 3 "" H 6600 3050 60  0001 C CNN
-	1    6600 3050
-	0    1    1    0
-$EndComp
-$Comp
-L power:VAA #PWR017
-U 1 1 5043CF97
-P 4100 3250
-F 0 "#PWR017" H 4100 3310 30  0001 C CNN
-F 1 "VAA" H 4100 3360 30  0000 C CNN
-F 2 "" H 4100 3250 60  0001 C CNN
-F 3 "" H 4100 3250 60  0001 C CNN
-	1    4100 3250
-	0    -1   -1   0
-$EndComp
-$Comp
 L Device:R R24
 U 1 1 503C490B
@@
 REF_IN
 $Comp
-L power:VCC #PWR059
-U 1 1 4FAECFB5
-P 7100 3950
-F 0 "#PWR059" H 7100 4050 30  0001 C CNN
-F 1 "VCC" H 7100 4050 30  0000 C CNN
-F 2 "" H 7100 3950 60  0001 C CNN
-F 3 "" H 7100 3950 60  0001 C CNN
-	1    7100 3950
-	1    0    0    -1
-$EndComp
-$Comp
 L Device:R R6
 U 1 1 4FAECFAE
@@
 $EndComp
 $Comp
-L power:VCC #PWR064
-U 1 1 4FAECE5B
-P 6900 3950
-F 0 "#PWR064" H 6900 4050 30  0001 C CNN
-F 1 "VCC" H 6900 4050 30  0000 C CNN
-F 2 "" H 6900 3950 60  0001 C CNN
-F 3 "" H 6900 3950 60  0001 C CNN
-	1    6900 3950
-	1    0    0    -1
-$EndComp
-$Comp
 L Device:R R5
 U 1 1 4FAECE50
@@
 $EndComp
 $Comp
-L power:VCC #PWR068
-U 1 1 4FAECBD8
-P 4700 7950
-F 0 "#PWR068" H 4700 8050 30  0001 C CNN
-F 1 "VCC" H 4700 8050 30  0000 C CNN
-F 2 "" H 4700 7950 60  0001 C CNN
-F 3 "" H 4700 7950 60  0001 C CNN
-	1    4700 7950
-	1    0    0    -1
-$EndComp
-$Comp
 L Device:C C6
 U 1 1 4FAECBBA
@@
 $EndComp
 $Comp
-L power:VCC #PWR078
-U 1 1 4FAA0C0D
-P 4100 2950
-F 0 "#PWR078" H 4100 3050 30  0001 C CNN
-F 1 "VCC" H 4100 3050 30  0000 C CNN
-F 2 "" H 4100 2950 60  0001 C CNN
-F 3 "" H 4100 2950 60  0001 C CNN
-	1    4100 2950
-	0    -1   -1   0
-$EndComp
-$Comp
 L power:GND #PWR079
 U 1 1 4FAA08EA
@@
 	1    0    0    -1
 $EndComp
-$Comp
-L power:VAA #PWR082
-U 1 1 5281BFB9
-P 7300 9800
-F 0 "#PWR082" H 7300 9860 30  0001 C CNN
-F 1 "VAA" H 7300 9910 30  0000 C CNN
-F 2 "" H 7300 9800 60  0001 C CNN
-F 3 "" H 7300 9800 60  0001 C CNN
-	1    7300 9800
-	1    0    0    -1
-$EndComp
 Wire Wire Line
 	7300 9800 7300 9900
@@
 	15850 7000 15550 7000
 $Comp
-L power:VAA #PWR090
-U 1 1 52EA1171
-P 15550 6900
-F 0 "#PWR090" H 15550 6960 30  0001 C CNN
-F 1 "VAA" H 15550 7010 30  0000 C CNN
-F 2 "" H 15550 6900 60  0001 C CNN
-F 3 "" H 15550 6900 60  0001 C CNN
-	1    15550 6900
-	1    0    0    -1
-$EndComp
-$Comp
 L power:GND #PWR091
 U 1 1 52EA1177
@@
 	4100 5600 4100 5500
 $Comp
-L power:VAA #PWR01
-U 1 1 50471BB9
-P 4400 4700
-F 0 "#PWR01" H 4400 4760 30  0001 C CNN
-F 1 "VAA" H 4400 4810 30  0000 C CNN
-F 2 "" H 4400 4700 60  0001 C CNN
-F 3 "" H 4400 4700 60  0001 C CNN
-	1    4400 4700
-	1    0    0    -1
-$EndComp
-$Comp
 L Device:L L3
 U 1 1 503BF2B7
@@
 Wire Wire Line
 	5300 5450 5300 5550
+$Comp
+L power:VAA #PWR0101
+U 1 1 606CFDC6
+P 6600 3050
+F 0 "#PWR0101" H 6600 2900 50  0001 C CNN
+F 1 "VAA" V 6617 3178 50  0000 L CNN
+F 2 "" H 6600 3050 50  0001 C CNN
+F 3 "" H 6600 3050 50  0001 C CNN
+	1    6600 3050
+	0    1    1    0
+$EndComp
+$Comp
+L power:VCC #PWR0102
+U 1 1 606D5D76
+P 6900 3950
+F 0 "#PWR0102" H 6900 3800 50  0001 C CNN
+F 1 "VCC" H 6917 4123 50  0000 C CNN
+F 2 "" H 6900 3950 50  0001 C CNN
+F 3 "" H 6900 3950 50  0001 C CNN
+	1    6900 3950
+	1    0    0    -1
+$EndComp
+$Comp
+L power:VCC #PWR0103
+U 1 1 606D914B
+P 7100 3950
+F 0 "#PWR0103" H 7100 3800 50  0001 C CNN
+F 1 "VCC" H 7117 4123 50  0000 C CNN
+F 2 "" H 7100 3950 50  0001 C CNN
+F 3 "" H 7100 3950 50  0001 C CNN
+	1    7100 3950
+	1    0    0    -1
+$EndComp
+$Comp
+L power:VCC #PWR0104
+U 1 1 606D9929
+P 4100 2950
+F 0 "#PWR0104" H 4100 2800 50  0001 C CNN
+F 1 "VCC" V 4118 3077 50  0000 L CNN
+F 2 "" H 4100 2950 50  0001 C CNN
+F 3 "" H 4100 2950 50  0001 C CNN
+	1    4100 2950
+	0    -1   -1   0
+$EndComp
+$Comp
+L power:VAA #PWR0105
+U 1 1 606DA38A
+P 4100 3250
+F 0 "#PWR0105" H 4100 3100 50  0001 C CNN
+F 1 "VAA" V 4118 3377 50  0000 L CNN
+F 2 "" H 4100 3250 50  0001 C CNN
+F 3 "" H 4100 3250 50  0001 C CNN
+	1    4100 3250
+	0    -1   -1   0
+$EndComp
+$Comp
+L power:VAA #PWR0106
+U 1 1 606DC211
+P 4400 4700
+F 0 "#PWR0106" H 4400 4550 50  0001 C CNN
+F 1 "VAA" H 4417 4873 50  0000 C CNN
+F 2 "" H 4400 4700 50  0001 C CNN
+F 3 "" H 4400 4700 50  0001 C CNN
+	1    4400 4700
+	1    0    0    -1
+$EndComp
+$Comp
+L power:VAA #PWR0107
+U 1 1 606E3B5E
+P 7300 9800
+F 0 "#PWR0107" H 7300 9650 50  0001 C CNN
+F 1 "VAA" H 7317 9973 50  0000 C CNN
+F 2 "" H 7300 9800 50  0001 C CNN
+F 3 "" H 7300 9800 50  0001 C CNN
+	1    7300 9800
+	1    0    0    -1
+$EndComp
+$Comp
+L power:VAA #PWR0108
+U 1 1 606E7DE5
+P 5650 7950
+F 0 "#PWR0108" H 5650 7800 50  0001 C CNN
+F 1 "VAA" H 5667 8123 50  0000 C CNN
+F 2 "" H 5650 7950 50  0001 C CNN
+F 3 "" H 5650 7950 50  0001 C CNN
+	1    5650 7950
+	1    0    0    -1
+$EndComp
+$Comp
+L power:VCC #PWR0109
+U 1 1 606EA95B
+P 4700 7950
+F 0 "#PWR0109" H 4700 7800 50  0001 C CNN
+F 1 "VCC" H 4717 8123 50  0000 C CNN
+F 2 "" H 4700 7950 50  0001 C CNN
+F 3 "" H 4700 7950 50  0001 C CNN
+	1    4700 7950
+	1    0    0    -1
+$EndComp
+$Comp
+L power:VAA #PWR0110
+U 1 1 606FA175
+P 10500 7900
+F 0 "#PWR0110" H 10500 7750 50  0001 C CNN
+F 1 "VAA" H 10517 8073 50  0000 C CNN
+F 2 "" H 10500 7900 50  0001 C CNN
+F 3 "" H 10500 7900 50  0001 C CNN
+	1    10500 7900
+	1    0    0    -1
+$EndComp
+$Comp
+L power:VAA #PWR0111
+U 1 1 606FB8F6
+P 15550 6900
+F 0 "#PWR0111" H 15550 6750 50  0001 C CNN
+F 1 "VAA" H 15567 7073 50  0000 C CNN
+F 2 "" H 15550 6900 50  0001 C CNN
+F 3 "" H 15550 6900 50  0001 C CNN
+	1    15550 6900
+	1    0    0    -1
+$EndComp
+$Comp
+L power:VAA #PWR0112
+U 1 1 606FDAE7
+P 12300 6100
+F 0 "#PWR0112" H 12300 5950 50  0001 C CNN
+F 1 "VAA" H 12317 6273 50  0000 C CNN
+F 2 "" H 12300 6100 50  0001 C CNN
+F 3 "" H 12300 6100 50  0001 C CNN
+	1    12300 6100
+	1    0    0    -1
+$EndComp
 $EndSCHEMATC
