File: hardware/hackrf-one/hackrf-one.kicad_pcb (KiCad board)
At the start: 4 copper layers, 120 x 75 mm, 432 parts, among them J1 USB-MICRO-B, J10 GND_CLIP, J2 RF-SHIELD-FRAME, J3 RF-SHIELD-COVER, J4 MOUNTING_HOLE, J5 MOUNTING_HOLE, J6 MOUNTING_HOLE, J7 MOUNTING_HOLE, J8 MOUNTING_HOLE, J9 MOUNTING_HOLE, P13 GPO1, P14 XCVR_CLKOUT, P15 INTR, P16 CLKIN, P17 GPO6, P18 OEB, P19 GPO3, P2 CLKOUT, P20 GPIO, P21 REF_IN, P22 I2S, P23 DBGEN, P24 TRST, P25 LPC_ISP, P26 LPC_JTAG, P27 MIXER_SDATA, P28 SD, P29 CPLD_JTAG, P3 GND, P30 BANK2_AUX, P31 MIXER_SCLK, P32 MIXER_ENX, P33 MIXER_RESETX, P34 MIX_BYPASS, P35 !MIX_BYPASS, P37 SCL, P38 SDA, P39 SSP1_SCK, P4 ANTENNA, P40 SSP1_COPI, P41 SSP1_CIPO, P42 TX, P43 RX, P44 HP, P45 LP, P46 TX_MIX_BP, P47 RX_MIX_BP, P48 TX_AMP, P49 RX_AMP, P5 LEDS, P50 AMP_BYPASS, P51 !TX_AMP_PWR, P52 !RX_AMP_PWR, P53 CS_XCVR, P54 CS_AD, P55 TXENABLE, P56 RXENABLE, P57 XTAL2, P58 GCK1, P59 GCK2, P6 GPO4, P60 SGPIO_CLK, P61 DA0, P62 DA7, P63 DD0, P64 DD9, P65 DA4, P66 DD5, P67 RSSI, P68 SPIFI_CS, P69 VREGMODE, P7 GPO2, P70 EN_1V8, P71 ID, P72 GP_CLKIN, P73 P1_2, P74 P1_1, P75 GP_CLKIN, P76 GP_CLKIN, P77 GP_CLKIN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

Commit message: HackRF One: update VBUS sense resistor values
Parts:
- R62: value 0 -> 10k
- R65: value 10k -> 18k
Changed lines of the file:
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@@
       (effects (font (size 0.4064 0.4064) (thickness 0.1016)))
     )
-    (fp_text value 0 (at 0 0.0508) (layer F.SilkS) hide
+    (fp_text value 10k (at 0 0.0508) (layer F.SilkS) hide
       (effects (font (size 0.4064 0.4064) (thickness 0.1016)))
     )
@@
       (effects (font (size 0.4064 0.4064) (thickness 0.1016)))
     )
-    (fp_text value 10k (at 0 0.0508 180) (layer F.SilkS) hide
+    (fp_text value 18k (at 0 0.0508 180) (layer F.SilkS) hide
       (effects (font (size 0.4064 0.4064) (thickness 0.1016)))
     )
