File: hardware/hackrf-one/mcu.sch (KiCad schematic (older format))
At the start: 134 parts, among them J1 USB-MICRO-B, P20 GPIO, P22 I2S, P23 DBGEN, P24 TRST, P25 LPC_ISP, P26 LPC_JTAG, P28 SD, P29 CPLD_JTAG, P3 GND, P30 BANK2_AUX, P5 LEDS, P68 SPIFI_CS, P69 VREGMODE, P70 EN_1V8, P71 ID, P72 GP_CLKIN, P73 P1_2, P74 P1_1, P75 GP_CLKIN, P76 GP_CLKIN, P77 GP_CLKIN, P78 GP_CLKIN, P79 GP_CLKIN, P80 SHIELD, P81 SPIFI_SIO2, P82 SPIFI_SIO3, Q5 MOSFET_P, SW1 DFU, SW2 RESET, U15 TVS, U20 W25Q80, U21 TPS62410, U23 LPC4320FBD144, U24 GSG-XC2C64A-7VQG100C, X2 MCU_XTAL, X3 RTC_XTAL

Commit message: HackRF One: update VBUS sense resistor values
Parts:
- R62: value 0 -> 10k; Description RES 0.0 OHM 1/16W 0402 SMD -> RES 10K OHM 1/16W 5% 0402 SMD; Part Number RMCF0402ZT0R00 -> RMCF0402JT10K0
- R65: value 10k -> 18k; Description RES 10K OHM 1/16W 5% 0402 SMD -> RES SMD 18K OHM 5% 1/16W 0402; Manufacturer Stackpole -> Yageo; Part Number RMCF0402JT10K0 -> RC0402JR-0718KL
Changed lines of the file:
@@
 AR Path="/5037043E/527F56E9" Ref="R62"  Part="1"
 F 0 "R62" V 3180 4000 50  0000 C CNN
-F 1 "0" V 3100 4000 50  0000 C CNN
+F 1 "10k" V 3100 4000 50  0000 C CNN
 F 2 "hackrf:GSG-0402" H 3100 4000 60  0001 C CNN
 F 3 "" H 3100 4000 60  0001 C CNN
 F 4 "Stackpole" H 3100 4000 60  0001 C CNN "Manufacturer"
-F 5 "RMCF0402ZT0R00" H 3100 4000 60  0001 C CNN "Part Number"
-F 6 "RES 0.0 OHM 1/16W 0402 SMD" H 3100 4000 60  0001 C CNN "Description"
+F 5 "RMCF0402JT10K0" H 3100 4000 60  0001 C CNN "Part Number"
+F 6 "RES 10K OHM 1/16W 5% 0402 SMD" H 3100 4000 60  0001 C CNN "Description"
 	1    3100 4000
 	-1   0    0    1
@@
 AR Path="/5037043E/527F56F2" Ref="R65"  Part="1"
 F 0 "R65" V 2980 4700 50  0000 C CNN
-F 1 "10k" V 2900 4700 50  0000 C CNN
+F 1 "18k" V 2900 4700 50  0000 C CNN
 F 2 "hackrf:GSG-0402" H 2900 4700 60  0001 C CNN
 F 3 "" H 2900 4700 60  0001 C CNN
-F 4 "Stackpole" H 2900 4700 60  0001 C CNN "Manufacturer"
-F 5 "RMCF0402JT10K0" H 2900 4700 60  0001 C CNN "Part Number"
-F 6 "RES 10K OHM 1/16W 5% 0402 SMD" H 2900 4700 60  0001 C CNN "Description"
+F 4 "Yageo" H 2900 4700 60  0001 C CNN "Manufacturer"
+F 5 "RC0402JR-0718KL" H 2900 4700 60  0001 C CNN "Part Number"
+F 6 "RES SMD 18K OHM 5% 1/16W 0402" H 2900 4700 60  0001 C CNN "Description"
 	1    2900 4700
 	-1   0    0    1
